Commit message: Add reliable Nav2 navigation simulation

File: differential_drive_robot_description/urdf/differential_drive_robot.urdf (robot description, URDF)
Before this commit: robot differential_drive_robot, 6 links, 5 joints
Links:
- added link imu_link, mass 0.02
Joints:
- added joint imu_joint: type fixed, parent base_link, child imu_link, origin xyz=0.09 0 0.08 rpy=0 0 0
